File: STM/STM32MP1/STM32MP135DAE7_MPU_HW/STM32MP135DAE7_MPU_HW.kicad_sch (KiCad schematic)
At the start: 0 parts

Commit message: h
Other:
- added sheet MPU_MEMORY_RAM (MPU_MEMORY_RAM.kicad_sch)
- added sheet MPU_MEMORY_STORAGE-NONVOLATILE (MPU_MEMORY_STORAGE-NONVOLATILE.kicad_sch)
- added sheet MPU_POWER (MPU_POWER.kicad_sch)
Changed lines of the file:
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@@
 (kicad_sch (version 20230121) (generator eeschema)
   (paper "A3")
+  (sheet (at 157.48 113.03) (size 82.55 62.23) (fields_autoplaced)
+    (stroke (width 0.1524) (type solid))
+    (fill (color 0 0 0 0.0000))
+    (property "Sheetname" "MPU_MEMORY_RAM" (at 157.48 112.3184 0)
+      (effects (font (size 1.27 1.27)) (justify left bottom))
+    )
+    (property "Sheetfile" "MPU_MEMORY_RAM.kicad_sch" (at 157.48 175.8446 0)
+      (effects (font (size 1.27 1.27)) (justify left top) hide)
+    )
+    (instances
+      (project "STM32MP135DAE7_MPU_HW"
+        (path "/ab0681b4-f474-44a3-a08a-fd6523012440" (page "2"))
+      )
+    )
+  )
+  (sheet (at 137.16 113.03) (size 12.7 62.23) (fields_autoplaced)
+    (stroke (width 0.1524) (type solid))
+    (fill (color 0 0 0 0.0000))
+    (property "Sheetname" "MPU_POWER" (at 137.16 112.3184 0)
+      (effects (font (size 1.27 1.27)) (justify left bottom))
+    )
+    (property "Sheetfile" "MPU_POWER.kicad_sch" (at 137.16 175.8446 0)
+      (effects (font (size 1.27 1.27)) (justify left top) hide)
+    )
+    (instances
+      (project "STM32MP135DAE7_MPU_HW"
+        (path "/ab0681b4-f474-44a3-a08a-fd6523012440" (page "4"))
+      )
+    )
+  )
+  (sheet (at 254 113.03) (size 40.64 63.5) (fields_autoplaced)
+    (stroke (width 0.1524) (type solid))
+    (fill (color 0 0 0 0.0000))
+    (property "Sheetname" "MPU_MEMORY_STORAGE-NONVOLATILE" (at 254 112.3184 0)
+      (effects (font (size 1.27 1.27)) (justify left bottom))
+    )
+    (property "Sheetfile" "MPU_MEMORY_STORAGE-NONVOLATILE.kicad_sch" (at 254 177.1146 0)
+      (effects (font (size 1.27 1.27)) (justify left top) hide)
+    )
+    (instances
+      (project "STM32MP135DAE7_MPU_HW"
+        (path "/ab0681b4-f474-44a3-a08a-fd6523012440" (page "3"))
+      )
+    )
+  )
   (sheet_instances
     (path "/" (page "1"))
