File: ALLWINNER/F1C100S_F1C200S_SoC/F1C100S_F1C200S_MPU_HW/F1C100S_F1C200S_MPU_HW.kicad_pcb (KiCad board)
At the start: 4 copper layers, 50 x 50 mm, 53 parts, among them J1 USB_C_Receptacle, J2 Micro_SD_Card_Det, J3 Conn_01x04, SW1 MCU_RESET, SW2 MCU_RESET, U1 F1C100s, U2 SRV05-4, Y1 24Mhz

Commit message: fg
Parts:
- removed Y1: 24Mhz, Crystal:Crystal_SMD_3225-4Pin_3.2x2.5mm
- added C11: 2u2, Capacitor_SMD:C_0402_1005Metric, F.Cu at (229.6, 88.0)
- added C14: 2u2, Capacitor_SMD:C_0402_1005Metric, F.Cu at (229.6, 90.0)
- added C15: 2u2, Capacitor_SMD:C_0402_1005Metric, F.Cu at (229.6, 92.0)
- added C16: 2u2, Capacitor_SMD:C_0402_1005Metric, F.Cu at (229.6, 94.0)
- added C17: 2u2, Capacitor_SMD:C_0402_1005Metric, F.Cu at (229.6, 95.9)
- added C18: 2u2, Capacitor_SMD:C_0402_1005Metric, F.Cu at (229.6, 97.9)
- added C19: 2u2, Capacitor_SMD:C_0402_1005Metric, F.Cu at (232.5, 88.0)
- added C20: 2u2, Capacitor_SMD:C_0402_1005Metric, F.Cu at (232.5, 90.0)
- added C21: 2u2, Capacitor_SMD:C_0402_1005Metric, F.Cu at (232.5, 92.0)
- added C22: 2u2, Capacitor_SMD:C_0402_1005Metric, F.Cu at (232.5, 94.0)
- added C23: 2u2, Capacitor_SMD:C_0402_1005Metric, F.Cu at (232.5, 95.9)
- added C24: 2u2, Capacitor_SMD:C_0402_1005Metric, F.Cu at (232.5, 97.9)
- added C25: 2u2, Capacitor_SMD:C_0402_1005Metric, F.Cu at (235.3, 88.0)
- added C26: 2u2, Capacitor_SMD:C_0402_1005Metric, F.Cu at (235.3, 90.0)
- added C28: 2u2, Capacitor_SMD:C_0402_1005Metric, F.Cu at (235.3, 92.0)
- added C29: 100n, Capacitor_SMD:C_0603_1608Metric_Pad1.08x0.95mm_HandSolder, F.Cu at (242.4, 104.6)
- added C32: 12p, Capacitor_SMD:C_0402_1005Metric, F.Cu at (235.3, 94.0)
- added C33: 12p, Capacitor_SMD:C_0402_1005Metric, F.Cu at (235.3, 95.9)
- added D4: D_Schottky, Diode_SMD:D_SMA_Handsoldering, F.Cu at (241.8, 96.1)
- added J4: USB_C_Receptacle, Connector_USB:USB_C_Receptacle_HRO_TYPE-C-31-M-12, F.Cu at (234.0, 82.4)
- added J5: Conn_01x04, Connector_PinHeader_2.54mm:PinHeader_1x04_P2.54mm_Vertical, F.Cu at (225.1, 106.6)
- added J6: AudioJack4_SwitchTR1, Z_mycustom_footprint_lib:PJ-316A-6A, F.Cu at (208.2, 110.2)
- added R25: 5k1, Resistor_SMD:R_0402_1005Metric, F.Cu at (241.3, 79.6)
- added R28: 390, Resistor_SMD:R_0603_1608Metric, F.Cu at (244.8, 77.8)
- added R29: 2k2, Resistor_SMD:R_0402_1005Metric, F.Cu at (241.3, 81.6)
- added R30: 2k2, Resistor_SMD:R_0402_1005Metric, F.Cu at (241.3, 83.5)
- added R31: 10k, Resistor_SMD:R_0402_1005Metric, F.Cu at (241.3, 85.5)
- added R4: 5k1, Resistor_SMD:R_0402_1005Metric, F.Cu at (241.3, 77.6)
- added RV1: 10k, Potentiometer_SMD:Potentiometer_Bourns_3314J_Vertical, F.Cu at (231.2, 102.7)
- added RV2: 10k, Potentiometer_SMD:Potentiometer_Bourns_3314J_Vertical, F.Cu at (237.2, 102.7)
- added SW3: MCU_RESET, SamacSys_Parts:PTS526SK15SMTR2LFS, F.Cu at (233.7, 110.6)
- added U3: PCF8563T, Package_SO:SOIC-8_3.9x4.9mm_P1.27mm, F.Cu at (243.0, 109.7)
- added U4: W25Q128JVS, Package_SO:SOIC-8_5.23x5.23mm_P1.27mm, F.Cu at (241.9, 90.4)
- added U5: SRV05-4, Package_TO_SOT_SMD:SOT-23-6, F.Cu at (242.8, 101.1)
- added U6: ESP32-S3-WROOM-1, Espressif:ESP32-S3-WROOM-1, F.Cu at (217.8, 93.2)
- added Y2: Crystal, Crystal:Crystal_SMD_3215-2Pin_3.2x1.5mm, F.Cu at (241.3, 114.5)
- C10, C9: value 1uF -> 2u2; footprint Capacitor_SMD:C_0402_1005Metric_Pad0.74x0.62mm_HandSolder -> Capacitor_SMD:C_0402_1005Metric
- C12: value 1u -> 2u2
- C13: value 10u -> 2u2; footprint Capacitor_SMD:C_0603_1608Metric -> Capacitor_SMD:C_0402_1005Metric
- C7, C8: value TBD -> 2u2; footprint Capacitor_SMD:C_0402_1005Metric_Pad0.74x0.62mm_HandSolder -> Capacitor_SMD:C_0402_1005Metric
- R26, R27: value 200K -> 5k1; footprint Resistor_SMD:R_0402_1005Metric_Pad0.72x0.64mm_HandSolder -> Resistor_SMD:R_0402_1005Metric
- moved U1 124.2 mm to (204.6, 124.3)
- moved FID1 55.4 mm to (178.3, 109.7)
- moved R14 55.4 mm to (185.6, 86.7)
- moved R15 55.4 mm to (185.6, 88.7)
- moved R16 55.4 mm to (185.6, 90.7)
- moved R17 55.4 mm to (185.6, 92.7)
- moved R18 55.4 mm to (185.6, 94.7)
- moved R19 55.4 mm to (185.6, 96.6)
- moved R20 55.4 mm to (185.6, 98.6)
- moved R21 55.4 mm to (188.5, 86.7)
- moved R22 55.4 mm to (188.5, 88.7)
- moved R23 55.4 mm to (188.5, 90.7)
- moved R24 55.4 mm to (188.5, 92.7)
- moved R26 55.4 mm to (178.7, 93.5)
- moved R27 55.4 mm to (178.7, 95.5)
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Connections:
- C10 pad 1: GND -> +3V3
- C10 pad 2: Net-(U1A-VRA2) -> GND
- C12 pad 1: +2V5 -> +3V3
- C7 pad 1: GND -> +3V3
- C7 pad 2: Net-(U1A-HOSCO) -> GND
- C8 pad 1: GND -> +3V3
- C8 pad 2: Net-(U1A-HOSCI) -> GND
- C9 pad 1: GND -> Net-(U1B-SVREF)
- C9 pad 2: Net-(U1A-VRA1) -> GND
- R23 pad 2: SDA -> SCL
- R24 pad 2: SCL -> SDA
- R26 pad 1: GND -> +3V3
- R26 pad 2: Net-(U1A-VRA1) -> /I2C1_SCL
- R27 pad 1: GND -> +3V3
- R27 pad 2: Net-(U1A-VRA2) -> /I2C1_SDA
- U1 pad 1: /AMP_HPL -> Net-(U1A-HPL)
- U1 pad 10: /USART1_TX -> unconnected-(U1A-PD4/LCD_D6/UART1_TX/EINTD4-Pad10)
- U1 pad 2: GND -> Net-(U1A-HPCOMFB)
- U1 pad 23: /I2C2_SCL -> unconnected-(U1A-PD15/LCD_D21/UART2_RTS/TWI2_SCK/EINTD15-Pad23)
- U1 pad 24: /I2C2_SDA -> unconnected-(U1A-PD16/LCD_D22/UART2_CTS/TWI2_SDA/EINTD16-Pad24)
- U1 pad 3: unconnected-(U1A-HPCOM-Pad3) -> Net-(U1A-HPCOM)
- U1 pad 33: unconnected-(U1B-SVREF-Pad33) -> Net-(U1B-SVREF)
- U1 pad 39: unconnected-(U1A-PE10/CSI_D7/UART2_CTS/SPI1_MISO/EINTE10-Pad39) -> /SPI1_MISO
- U1 pad 40: unconnected-(U1A-PE9/CSI_D6/UART2_RTS/SPI1_CLK/EINTE9-Pad40) -> /SPI1_CLK
- U1 pad 41: unconnected-(U1A-PE8/CSI_D5/UART2_RX/SPI1_MOSI/EINTE8-Pad41) -> /SPI1_MOSI
- U1 pad 42: unconnected-(U1A-PE7/CSI_D4/UART2_TX/SPI1_CS/EINTE7-Pad42) -> /SPI1_CS
- U1 pad 48: unconnected-(U1A-PE1/CSI_VSYNC/LCD_D1/TWI2_SDA/UART0_TX/EINTE1-Pad48) -> UART0_TX
- U1 pad 49: unconnected-(U1A-PE0/CSI_HSYNC/LCD_D0/TWI2_SCK/UART0_RX/EINTE0-Pad49) -> UART0_RX
- U1 pad 51: Net-(U1A-HOSCI) -> unconnected-(U1A-HOSCI-Pad51)
- U1 pad 52: Net-(U1A-HOSCO) -> unconnected-(U1A-HOSCO-Pad52)
- U1 pad 6: /WIFI_INT -> unconnected-(U1A-PD0/LCD_D2/TWI0_SDA/RSB_SDA/EINTD0-Pad6)
- U1 pad 63: /SPI1_MISO -> unconnected-(U1A-TPY2-Pad63)
- U1 pad 64: /SPI1_CLK -> unconnected-(U1A-TPY1-Pad64)
- U1 pad 65: /SPI1_MOSI -> unconnected-(U1A-TPX2-Pad65)
- U1 pad 66: /SPI1_CS -> unconnected-(U1A-TPX1-Pad66)
- U1 pad 7: /WIFI_RESET -> unconnected-(U1A-PD1/LCD_D3/UART1_RTS/EINTD1-Pad7)
- U1 pad 8: /TOUCH_INT -> unconnected-(U1A-PD2/LCD_D4/UART1_CTS/EINTD2-Pad8)
- U1 pad 81: Net-(U1A-VRA1) -> /VRA1
- U1 pad 83: Net-(U1A-VRA2) -> /VRA2
- U1 pad 84: unconnected-(U1A-FMINL-Pad84) -> Net-(U1A-FMINL)
- U1 pad 85: unconnected-(U1A-FMINR-Pad85) -> Net-(U1A-FMINR)
- U1 pad 86: unconnected-(U1A-LINL-Pad86) -> Net-(U1A-LINL)
- U1 pad 87: unconnected-(U1A-MICIN-Pad87) -> Net-(U1A-MICIN)
- U1 pad 88: /AMP_HPR -> Net-(U1A-HPR)
- U1 pad 9: /USART1_RX -> unconnected-(U1A-PD3/LCD_D5/UART1_RX/EINTD3-Pad9)
Routing:
- added copper zone on F.Cu, net GND
- added copper zone on In1.Cu, net GND
- added copper zone on In2.Cu, net GND
Other:
- board size 50 x 50 mm -> 100 x 100 mm
