File: ALLWINNER/F1C100S_F1C200S_SoC/F1C100S_F1C200S_MPU_HW/F1C100S_F1C200S_MPU_HW.kicad_sch (KiCad schematic)
At the start: 67 parts, among them J1 USB_C_Receptacle, J2 Micro_SD_Card_Det, J3 Conn_01x04, SW1 MCU_RESET, SW2 MCU_RESET, U1 F1C100s, U2 SRV05-4, Y2 24Mhz

Commit message: fg
Parts:
- removed C25, C26: TBD, Capacitor_SMD:C_0402_1005Metric_Pad0.74x0.62mm_HandSolder, symbol Device:C
- removed C40, C41: 1uF, Capacitor_SMD:C_0402_1005Metric_Pad0.74x0.62mm_HandSolder, symbol Device:C
- removed R30, R31: 200K, Resistor_SMD:R_0402_1005Metric_Pad0.72x0.64mm_HandSolder, symbol Device:R
- removed Y2: 24Mhz, Crystal:Crystal_SMD_3225-4Pin_3.2x2.5mm, symbol Device:Crystal_GND24
- added C10, C26, C28, C7, C8, C9: 2u2, Capacitor_SMD:C_0402_1005Metric, symbol Device:C_Small
- added C27: 1-3F, symbol Device:C_Polarized_Small
- added C29: 100n, Capacitor_SMD:C_0603_1608Metric_Pad1.08x0.95mm_HandSolder, symbol Device:C_Small
- added C32, C33: 12p, Capacitor_SMD:C_0402_1005Metric, symbol Device:C_Small
- added D4: D_Schottky, Diode_SMD:D_SMA_Handsoldering, symbol Device:D_Schottky
- added J4: USB_C_Receptacle, Connector_USB:USB_C_Receptacle_HRO_TYPE-C-31-M-12, symbol Connector:USB_C_Receptacle
- added J5: Conn_01x04, Connector_PinHeader_2.54mm:PinHeader_1x04_P2.54mm_Vertical, symbol Connector_Generic:Conn_01x04
- added J6: AudioJack4_SwitchTR1, Z_mycustom_footprint_lib:PJ-316A-6A, symbol Connector:AudioJack4_SwitchTR1
- added R25, R26, R27, R4: 5k1, Resistor_SMD:R_0402_1005Metric, symbol Device:R_Small
- added R28: 390, Resistor_SMD:R_0603_1608Metric, symbol Device:R_Small
- added R29, R30: 2k2, Resistor_SMD:R_0402_1005Metric, symbol Device:R_Small
- added R31: 10k, Resistor_SMD:R_0402_1005Metric, symbol Device:R_Small
- added RV1, RV2: 10k, Potentiometer_SMD:Potentiometer_Bourns_3314J_Vertical, symbol Device:R_Potentiometer
- added SW3: MCU_RESET, SamacSys_Parts:PTS526SK15SMTR2LFS, symbol Switch:SW_SPST
- added TP2, TP3, TP4, TP5, TP6: TestPoint, TestPoint:TestPoint_Pad_1.0x1.0mm, symbol Connector:TestPoint
- added U3: PCF8563T, Package_SO:SOIC-8_3.9x4.9mm_P1.27mm, symbol Timer_RTC:PCF8563T
- added U4: W25Q128JVS, Package_SO:SOIC-8_5.23x5.23mm_P1.27mm, symbol Memory_Flash:W25Q128JVS
- added U5: SRV05-4, Package_TO_SOT_SMD:SOT-23-6, symbol Power_Protection:SRV05-4
- added U6: ESP32-S3-WROOM-1, Espressif:ESP32-S3-WROOM-1, symbol Espressif:ESP32-S3-WROOM-1
- added Y2: Crystal, Crystal:Crystal_SMD_3215-2Pin_3.2x1.5mm, symbol Device:Crystal
- C12: value 1u -> 2u2; LCSC C52923 -> C12530
Connections:
- net +2V5: now also R30.1
- net +3V3: now also C12.1, C10.1, C28.1, C7.1, C8.1, J5.4 (Pin_4), R26.1, R27.1, R31.1, RV1.3, RV2.1, U4.8 (VCC), U6.2 (3V3)
- net +5V: now also R28.2
- net ESP_BOOT: now also U6.27 (GPIO0/BOOT)
- net GND: now also C10.2, C26.2, C27.2, C28.2, C29.2, C32.2, C33.2, C7.2, C8.2, C9.2, J4.A1 (GND), J4.A12 (GND), J4.B1 (GND), J4.B12 (GND), J5.1 (Pin_1), R25.2, R29.1, R4.2, RV1.1, RV2.3, SW3.2 (B), U3.4 (VSS), U4.4 (GND), U5.2 (VN), U6.1 (GND), U6.40 (GND), U6.41 (GND); no longer U1.2 (HPCOMFB)
- net I2C1_SCL: now also J5.3 (Pin_3), R26.2
- net I2C1_SDA: now also J5.2 (Pin_2), R27.2
- net SCL: now also R23.2, U3.6 (SCL); no longer R24.2
- net SDA: now also R24.2, U3.5 (SDA); no longer R23.2
- net SPI1_CLK: now also U1.40 (PE9/CSI_D6/UART2_RTS/SPI1_CLK/EINTE9), U4.6 (CLK); no longer U1.64 (TPY1)
- net SPI1_CS: now also U1.42 (PE7/CSI_D4/UART2_TX/SPI1_CS/EINTE7), U4.1 (~{CS}); no longer U1.66 (TPX1)
- net SPI1_MISO: now also U1.39 (PE10/CSI_D7/UART2_CTS/SPI1_MISO/EINTE10), U4.2 (DO(IO1)); no longer U1.63 (TPY2)
- net SPI1_MOSI: now also U1.41 (PE8/CSI_D5/UART2_RX/SPI1_MOSI/EINTE8), U4.5 (DI(IO0)); no longer U1.65 (TPX2)
- net VBUS: now also J4.A4 (VBUS), J4.A9 (VBUS), J4.B4 (VBUS), J4.B9 (VBUS), U5.5 (VP)
- net at U1.33 (SVREF): now also C9.1, R29.2, R30.2
- net VRA1: now reaches U1.81 (VRA1)
- net VRA1: now also RV1.2
- net at U1.3 (HPCOM): now also J6.R2
- net UART0_TX: now reaches U1.48 (PE1/CSI_VSYNC/LCD_D1/TWI2_SDA/UART0_TX/EINTE1)
- net UART0_RX: now reaches U1.49 (PE0/CSI_HSYNC/LCD_D0/TWI2_SCK/UART0_RX/EINTE0)
- net VRA2: now reaches U1.83 (VRA2)
- net VRA2: now also RV2.2
- net at U1.84 (FMINL): now also TP3.1
- net at U1.85 (FMINR): now also TP2.1
- net at U1.86 (LINL): now also TP4.1
- net at U1.87 (MICIN): now also J6.S
- net AMP_HPL: no longer names the net of U1.1 (HPL)
- net AMP_HPL: now also J6.T
- net AMP_HPR: no longer names the net of U1.88 (HPR)
- net AMP_HPR: now also J6.R1
- net I2C2_SCL: no longer names the net of U1.23 (PD15/LCD_D21/UART2_RTS/TWI2_SCK/EINTD15)
- net I2C2_SDA: no longer names the net of U1.24 (PD16/LCD_D22/UART2_CTS/TWI2_SDA/EINTD16)
- net TOUCH_INT: no longer names the net of U1.8 (PD2/LCD_D4/UART1_CTS/EINTD2)
- net USART1_RX: no longer names the net of U1.9 (PD3/LCD_D5/UART1_RX/EINTD3)
- net USART1_TX: no longer names the net of U1.10 (PD4/LCD_D6/UART1_TX/EINTD4)
- net WIFI_INT: no longer names the net of U1.6 (PD0/LCD_D2/TWI0_SDA/RSB_SDA/EINTD0)
- net WIFI_RESET: no longer names the net of U1.7 (PD1/LCD_D3/UART1_RTS/EINTD1)
- new net: C33.1, U3.1 (OSCI), Y2.1
- new net: C26.1, C27.1, D4.1 (K), U3.8 (VDD)
- new net: TP5.1, U1.2 (HPCOMFB)
- new net: J6.TN, TP6.1
- new net: C32.1, U3.2 (OSCO), Y2.2
- new net: D4.2 (A), R28.1
- new net D1-: J4.A7 (D-), J4.B7 (D-), U5.6 (IO4), U6.13 (GPIO19/U1RTS/ADC2_CH8/CLK_OUT2/USB_D-)
- new net D2+: J4.A6 (D+), J4.B6 (D+), U5.1 (IO1), U6.14 (GPIO20/U1CTS/ADC2_CH9/CLK_OUT1/USB_D+)
- new net ESP_EN: C29.1, R31.2, SW3.1 (A), U6.3 (EN)
- new net cc1_1: J4.A5 (CC1), R4.1
- new net cc2_1: J4.B5 (CC2), R25.1
- no-connect marks 13 -> 25
Other:
- note added: "USB2 ESP32"
- note removed: "I2C"
- note removed: "I2C2"
- note removed: "LCD SPI1"
- note removed: "M-BUS"
- note removed: "On Board"
- note removed: "USART1"
- moved on the sheet: C1, C2, C3, D1, D2, D3, FB1, FID1, FID2, FID3, J1, R1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
